Commit message: Adapt kinova stack for JDX challenge

File: kinova_description/urdf/kinova_inertial.xacro (robot description, xacro)
@@ -85,5 +85,5 @@
   <xacro:unless value="${mesh_no-4}">
     <inertial>
-        <mass value="0.426367" />
+        <mass value="0.1785" />
         <origin xyz="0 -0.037 -0.0642" />
         <xacro:inertia_cylinder height="0.02"  radius = "0.04" mass="0.1785"/>
@@ -141,5 +141,5 @@
   <xacro:unless value="${mesh_no - 55}">
     <inertial>
-        <mass value="0.99" />
+        <mass value="0.727" />
         <origin xyz="0 0 -0.06" />
         <xacro:inertia_cylinder height="0.03"  radius = "0.04" mass="0.727"/>
